File: Projeto Eagle/Versão conector/FIO_M.sch (EAGLE design)
At the start: 4 parts, among them J1 CONECTOR

Commit message: correção de pads e adição de label de versionamento
Parts:
- J1: value CONECTOR -> CONECTOR_MACHO; device Eletroblocks Lib:CONECTOR -> Eletroblocks Lib:CONECTOR_MACHO
- renumbered U$2 to J3
Changed lines of the file:
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@@
 <layer number="91" name="Nets" color="2" fill="1" visible="yes" active="yes"/>
 <layer number="92" name="Busses" color="1" fill="1" visible="yes" active="yes"/>
-<layer number="93" name="Pins" color="2" fill="1" visible="no" active="yes"/>
+<layer number="93" name="Pins" color="2" fill="1" visible="yes" active="yes"/>
 <layer number="94" name="Symbols" color="4" fill="1" visible="yes" active="yes"/>
 <layer number="95" name="Names" color="7" fill="1" visible="yes" active="yes"/>
@@
 </classes>
 <parts>
-<part name="J1" library="Eletroblocks Lib" deviceset="CONECTOR" device="" override_package3d_urn="urn:adsk.eagle:package:23100835/3" override_package_urn="urn:adsk.eagle:footprint:23100837/1"/>
+<part name="J1" library="Eletroblocks Lib" deviceset="CONECTOR_MACHO" device="" override_package3d_urn="urn:adsk.eagle:package:23100835/3" override_package_urn="urn:adsk.eagle:footprint:23100837/1" override_locally_modified="yes"/>
 <part name="U$1" library="Eletroblocks Lib" deviceset="PAD" device=""/>
-<part name="U$2" library="Eletroblocks Lib" deviceset="PAD" device="" override_package3d_urn="urn:adsk.eagle:package:23100844/2" override_package_urn="urn:adsk.eagle:footprint:23100847/1"/>
+<part name="J3" library="Eletroblocks Lib" deviceset="PAD" device="" override_package3d_urn="urn:adsk.eagle:package:23100844/2" override_package_urn="urn:adsk.eagle:footprint:23100847/1" override_locally_modified="yes"/>
 <part name="VCC" library="Eletroblocks Lib" deviceset="PAD" device=""/>
 </parts>
@@
 </instance>
 <instance part="U$1" gate="G$1" x="21.59" y="104.61" smashed="yes"/>
-<instance part="U$2" gate="G$1" x="21.51" y="100.58" smashed="yes"/>
+<instance part="J3" gate="G$1" x="21.51" y="100.58" smashed="yes"/>
 <instance part="VCC" gate="G$1" x="21.39" y="96.68" smashed="yes"/>
 </instances>
@@
 <pinref part="J1" gate="G$1" pin="2"/>
 <wire x1="4.52" y1="100.65" x2="4.52" y2="100.61" width="0.1524" layer="91"/>
-<pinref part="U$2" gate="G$1" pin="P$1"/>
+<pinref part="J3" gate="G$1" pin="P$1"/>
 <wire x1="4.52" y1="100.65" x2="21.57" y2="100.65" width="0.1524" layer="91"/>
 <wire x1="21.57" y1="100.65" x2="21.51" y2="100.58" width="0.1524" layer="91"/>
